File: BPS/Debugger/Debugger/file5C5F7A4C.sch (KiCad schematic (older format))
At the start: 23 parts, among them J2 CAN_Out, U3 ADM3055E, U4 CDSOT23-T24CAN

Commit message: NC flags, 3.3v flag, etc.
Parts:
- J2: symbol utsvt-connectors:CANConnector -> Debugger-rescue:CANConnector-utsvt-connectors
- U3: symbol utsvt-chips:ADM3055E -> Debugger-rescue:ADM3055E-utsvt-chips
- U4: symbol utsvt-chips:CDSOT23-T24CAN -> Debugger-rescue:CDSOT23-T24CAN-utsvt-chips
Changed lines of the file:
@@
 $EndComp
 $Comp
-L utsvt-chips:ADM3055E U3
+L Debugger-rescue:ADM3055E-utsvt-chips U3
 U 1 1 5C5F8645
 P 4050 3400
@@
 	7350 2700 7650 2700
 $Comp
-L utsvt-chips:CDSOT23-T24CAN U4
+L Debugger-rescue:CDSOT23-T24CAN-utsvt-chips U4
 U 1 1 5C63851C
 P 8000 2750
@@
 $EndComp
 $Comp
-L utsvt-connectors:CANConnector J2
+L Debugger-rescue:CANConnector-utsvt-connectors J2
 U 1 1 5C648177
 P 9050 3600
