File: BPS/Debugger/Debugger/_autosave-Debugger.kicad_pcb (KiCad board)
At the start: 2 copper layers, 66 parts, among them J1 Conn_01x03, J2 CAN_Out, J3 Barrel_Jack, SW1 Switch:SW_Push, U1 STM32F413RHTx, U2 NCP1117-3.3_SOT223, U3 ADM3055E, U4 CDSOT23-T24CAN, U5 LD1117S33TR_SOT223, U6 RI3-1205S, Y1 Crystal

Commit message: debugger
Parts:
- moved U2 161.4 mm to (62.2, 68.6)
- moved J1 107.5 mm to (128.3, 102.9)
- moved JP1 67.1 mm to (256.5, 110.5)
- moved C2 35.3 mm to (166.4, 24.1)
- moved C16 11.5 mm to (220.6, 95.2)
- moved C17 11.5 mm to (209.6, 95.2)
- moved R3 11.5 mm to (213.4, 95.2)
- moved C19 11.5 mm to (217.2, 95.2)
- moved C20 11.5 mm to (225.7, 95.2)
- moved C14 10.3 mm to (223.5, 90.2)
- moved C3 9.92 mm to (182.5, 24.1)
- moved TP4 8.13 mm to (212.1, 62.2)
- moved R1 6.48 mm to (213.4, 86.4)
- moved R2 6.48 mm to (216.8, 86.4)
- moved TP6 5.24 mm to (199.4, 62.2)
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