File: BPS/Master/SPI.sch (KiCad schematic (older format))
At the start: 51 parts, among them J10 DisplayJumper, J7 VoltageSlaveConnector, J8 DisplayConnector, J9 TempSlaveConnector, U10 LTC6820, U11 HX1188FNL, U12 LTC6820, U13 Si8641EC-B-IS1, U14 SI8660EC-B-IS1, U15 RI3-1205S

Commit message: Edited inductor choke in BPS master.
Parts:
- L4: footprint Inductor_SMD:L_0805_2012Metric -> UTSVT_BPS:SRF0905A; symbol Device:L -> utsvt-bps:SRF0905-100Y
Connections:
- wire segments 225 -> 233
Other:
- moved on the sheet: C47
Changed lines of the file:
@@
 L power:+12V #PWR?
 U 1 1 5C3DD0E6
-P 2600 7000
+P 1900 7000
 AR Path="/5C29E573/5C3DD0E6" Ref="#PWR?"  Part="1"
 AR Path="/5C4C7509/5C3DD0E6" Ref="#PWR0108"  Part="1"
-F 0 "#PWR0108" H 2600 6850 50  0001 C CNN
-F 1 "+12V" H 2615 7173 50  0000 C CNN
-F 2 "" H 2600 7000 50  0001 C CNN
-F 3 "" H 2600 7000 50  0001 C CNN
-	1    2600 7000
-	1    0    0    -1
-$EndComp
-Wire Wire Line
-	2600 7450 2600 7500
+F 0 "#PWR0108" H 1900 6850 50  0001 C CNN
+F 1 "+12V" H 1915 7173 50  0000 C CNN
+F 2 "" H 1900 7000 50  0001 C CNN
+F 3 "" H 1900 7000 50  0001 C CNN
+	1    1900 7000
+	1    0    0    -1
+$EndComp
+Wire Wire Line
+	1900 7450 1900 7500
 $Comp
 L Device:C C?
 U 1 1 5C3DD0EE
-P 2850 7250
+P 2150 7250
 AR Path="/5C29E573/5C3DD0EE" Ref="C?"  Part="1"
 AR Path="/5C4C7509/5C3DD0EE" Ref="C47"  Part="1"
-F 0 "C47" H 2968 7296 50  0000 L CNN
-F 1 "4.7uF" H 2968 7205 50  0000 L CNN
-F 2 "Capacitor_SMD:C_0805_2012Metric" H 2888 7100 50  0001 C CNN
-F 3 "~" H 2850 7250 50  0001 C CNN
-	1    2850 7250
-	1    0    0    -1
-$EndComp
-Wire Wire Line
-	2600 7450 2850 7450
-$Comp
-L Device:L L?
+F 0 "C47" H 2268 7296 50  0000 L CNN
+F 1 "4.7uF" H 2268 7205 50  0000 L CNN
+F 2 "Capacitor_SMD:C_0805_2012Metric" H 2188 7100 50  0001 C CNN
+F 3 "~" H 2150 7250 50  0001 C CNN
+	1    2150 7250
+	1    0    0    -1
+$EndComp
+Wire Wire Line
+	1900 7450 2150 7450
+$Comp
+L utsvt-bps:SRF0905-100Y L?
 U 1 1 5C3DD0F6
-P 3150 7050
+P 2400 7000
 AR Path="/5C29E573/5C3DD0F6" Ref="L?"  Part="1"
 AR Path="/5C4C7509/5C3DD0F6" Ref="L4"  Part="1"
-F 0 "L4" V 3340 7050 50  0000 C CNN
-F 1 "10uH" V 3249 7050 50  0000 C CNN
-F 2 "Inductor_SMD:L_0805_2012Metric" H 3150 7050 50  0001 C CNN
-F 3 "~" H 3150 7050 50  0001 C CNN
-	1    3150 7050
-	0    -1   -1   0
-$EndComp
-Wire Wire Line
-	2600 7000 2600 7050
-Wire Wire Line
-	2600 7050 2850 7050
-Wire Wire Line
-	2850 7100 2850 7050
-Connection ~ 2850 7050
-Wire Wire Line
-	2850 7050 3000 7050
-Wire Wire Line
-	2850 7400 2850 7450
-Connection ~ 2850 7450
-Wire Wire Line
-	2850 7450 3450 7450
-Wire Wire Line
-	3450 7050 3300 7050
+F 0 "L4" H 2650 7250 50  0000 C CNN
+F 1 "10uH" H 2700 7150 50  0000 C CNN
+F 2 "UTSVT_BPS:SRF0905A" H 2400 7000 50  0001 C CNN
+F 3 "~" H 2400 7000 50  0001 C CNN
+	1    2400 7000
+	1    0    0    -1
+$EndComp
+Wire Wire Line
+	1900 7000 1900 7050
+Wire Wire Line
+	1900 7050 2150 7050
+Wire Wire Line
+	2150 7100 2150 7050
+Connection ~ 2150 7050
+Wire Wire Line
+	2150 7400 2150 7450
+Connection ~ 2150 7450
 Wire Wire Line
 	4650 7450 4650 7350
@@
 L power:GNDPWR #PWR?
 U 1 1 5C3DD13C
-P 2600 7500
+P 1900 7500
 AR Path="/5C29E573/5C3DD13C" Ref="#PWR?"  Part="1"
 AR Path="/5C4C7509/5C3DD13C" Ref="#PWR0111"  Part="1"
-F 0 "#PWR0111" H 2600 7300 50  0001 C CNN
-F 1 "GNDPWR" H 2604 7346 50  0000 C CNN
-F 2 "" H 2600 7450 50  0001 C CNN
-F 3 "" H 2600 7450 50  0001 C CNN
-	1    2600 7500
+F 0 "#PWR0111" H 1900 7300 50  0001 C CNN
+F 1 "GNDPWR" H 1904 7346 50  0000 C CNN
+F 2 "" H 1900 7450 50  0001 C CNN
+F 3 "" H 1900 7450 50  0001 C CNN
+	1    1900 7500
 	1    0    0    -1
 $EndComp
@@
 Wire Wire Line
 	10550 4250 10100 4250
+Wire Wire Line
+	2150 7450 3450 7450
+Wire Wire Line
+	3250 7050 3250 7000
+Wire Wire Line
+	3250 7000 3200 7000
+Wire Wire Line
+	3250 7050 3450 7050
+Wire Wire Line
+	3200 7100 3250 7100
+Wire Wire Line
+	3250 7100 3250 7050
+Connection ~ 3250 7050
+Wire Wire Line
+	2400 7100 2350 7100
+Wire Wire Line
+	2350 7100 2350 7050
+Wire Wire Line
+	2350 7000 2400 7000
+Wire Wire Line
+	2150 7050 2350 7050
 Wire Bus Line
 	6350 5400 6350 6000
+Connection ~ 2350 7050
+Wire Wire Line
+	2350 7050 2350 7000
 $EndSCHEMATC
