File: BPS/Master/CAN.sch (KiCad schematic (older format))
At the start: 23 parts, among them J5 CAN_Out, U4 CDSOT23-T24CAN, U5 ADM3055E

Commit message: Adds master board v1.1.
Parts:
- removed TP5: CAN_ISO_Vout, TestPoint:TestPoint_Keystone_5005-5009_Compact, symbol Connector:TestPoint
- removed TP6: CAN_ISO_Vin, TestPoint:TestPoint_Keystone_5005-5009_Compact, symbol Connector:TestPoint
- removed TP7: CAN_ISO_GndIn, TestPoint:TestPoint_Keystone_5005-5009_Compact, symbol Connector:TestPoint
- removed TP8: CAN_ISO_GndOut, TestPoint:TestPoint_Keystone_5005-5009_Compact, symbol Connector:TestPoint
- J8: renamed from J5; symbol utsvt-connectors:CANConnector -> BPSMaster-rescue:CANConnector-utsvt-connectors
- U12: renamed from U4; symbol utsvt-chips:CDSOT23-T24CAN -> BPSMaster-rescue:CDSOT23-T24CAN-utsvt-chips
- U13: renamed from U5; symbol utsvt-chips:ADM3055E -> BPSMaster-rescue:ADM3055E-utsvt-chips
- renumbered C19 to C29, C20 to C30, C21 to C31, C22 to C32, C23 to C33, C24 to C34, C25 to C35, C26 to C36, L2 to L3, L3 to L4, R2 to R41, R3 to R42, R4 to R43, TP9 to TP7, TP12 to TP8
Connections:
- wire segments 104 -> 94
Other:
- note added: "As long as total equals to 120 Ohms,\nthe two termination resistors can be any value"
Changed lines of the file:
@@
 EESchema Schematic File Version 4
 LIBS:BPSMaster-cache
-EELAYER 29 0
+EELAYER 30 0
 EELAYER END
 $Descr A4 11693 8268
 encoding utf-8
-Sheet 3 7
+Sheet 8 11
 Title ""
 Date ""
@@
 $EndDescr
 $Comp
-L utsvt-connectors:CANConnector J5
+L BPSMaster-rescue:CANConnector-utsvt-connectors J8
 U 1 1 5C2B42F3
 P 9250 3800
-F 0 "J5" H 9250 3550 60  0000 C CNN
+F 0 "J8" H 9250 3550 60  0000 C CNN
 F 1 "CAN_Out" H 9250 4050 60  0000 C CNN
 F 2 "UTSVT_Connectors:Molex_MicroFit3.0_1x4xP3.00mm_PolarizingPeg_Vertical" H 9400 4100 60  0001 C CNN
@@
 $EndComp
 $Comp
-L Device:R R3
+L Device:R R42
 U 1 1 5C2B42FA
 P 8200 3550
-F 0 "R3" V 8280 3550 50  0000 C CNN
+F 0 "R42" V 8280 3550 50  0000 C CNN
 F 1 "60" V 8200 3550 50  0000 C CNN
 F 2 "Resistor_SMD:R_0805_2012Metric" V 8130 3550 50  0001 C CNN
@@
 $EndComp
 $Comp
-L Device:R R2
+L Device:R R41
 U 1 1 5C2B4301
 P 8000 3550
-F 0 "R2" V 8080 3550 50  0000 C CNN
+F 0 "R41" V 8080 3550 50  0000 C CNN
 F 1 "60" V 8000 3550 50  0000 C CNN
 F 2 "Resistor_SMD:R_0805_2012Metric" V 7930 3550 50  0001 C CNN
@@
 $EndComp
 $Comp
-L Device:C_Small C23
+L Device:C_Small C33
 U 1 1 5C2B4310
 P 2150 3350
-F 0 "C23" H 2160 3420 50  0000 L CNN
+F 0 "C33" H 2160 3420 50  0000 L CNN
 F 1 "10uF" H 2160 3270 50  0000 L CNN
 F 2 "Capacitor_SMD:C_0805_2012Metric" H 2150 3350 50  0001 C CNN
@@
 $EndComp
 $Comp
-L Device:C_Small C24
+L Device:C_Small C34
 U 1 1 5C2B4317
 P 2500 3350
-F 0 "C24" H 2510 3420 50  0000 L CNN
+F 0 "C34" H 2510 3420 50  0000 L CNN
 F 1 "0.1uF" H 2510 3270 50  0000 L CNN
 F 2 "Capacitor_SMD:C_0805_2012Metric" H 2500 3350 50  0001 C CNN
@@
 $EndComp
 $Comp
-L Device:C_Small C25
+L Device:C_Small C35
 U 1 1 5C2B431E
 P 2950 3350
-F 0 "C25" H 2960 3420 50  0000 L CNN
+F 0 "C35" H 2960 3420 50  0000 L CNN
 F 1 "0.1uF" H 2960 3270 50  0000 L CNN
 F 2 "Capacitor_SMD:C_0805_2012Metric" H 2950 3350 50  0001 C CNN
@@
 $EndComp
 $Comp
-L Device:C_Small C26
+L Device:C_Small C36
 U 1 1 5C2B4325
 P 3300 3350
-F 0 "C26" H 3310 3420 50  0000 L CNN
+F 0 "C36" H 3310 3420 50  0000 L CNN
 F 1 "0.01uF" H 3310 3270 50  0000 L CNN
 F 2 "Capacitor_SMD:C_0805_2012Metric" H 3300 3350 50  0001 C CNN
@@
 $EndComp
 $Comp
-L Device:C_Small C20
+L Device:C_Small C30
 U 1 1 5C2B432E
 P 6150 3200
-F 0 "C20" H 6160 3270 50  0000 L CNN
+F 0 "C30" H 6160 3270 50  0000 L CNN
 F 1 "10uF" H 6160 3120 50  0000 L CNN
 F 2 "Capacitor_SMD:C_0805_2012Metric" H 6150 3200 50  0001 C CNN
@@
 $EndComp
 $Comp
-L Device:C_Small C19
+L Device:C_Small C29
 U 1 1 5C2B4335
 P 5750 3200
-F 0 "C19" H 5760 3270 50  0000 L CNN
+F 0 "C29" H 5760 3270 50  0000 L CNN
 F 1 "0.22uF" H 5760 3120 50  0000 L CNN
 F 2 "Capacitor_SMD:C_0805_2012Metric" H 5750 3200 50  0001 C CNN
@@
 $EndComp
 $Comp
-L Device:Ferrite_Bead_Small L2
+L Device:Ferrite_Bead_Small L3
 U 1 1 5C2B433C
 P 5950 3050
-F 0 "L2" V 5850 3100 50  0000 L CNN
+F 0 "L3" V 5850 3100 50  0000 L CNN
 F 1 "2kH" V 5850 2900 50  0000 L CNN
 F 2 "Inductor_SMD:L_0805_2012Metric" V 5880 3050 50  0001 C CNN
@@
 $EndComp
 $Comp
-L Device:Ferrite_Bead_Small L3
+L Device:Ferrite_Bead_Small L4
 U 1 1 5C2B4343
 P 5950 3350
-F 0 "L3" V 6050 3400 50  0000 L CNN
+F 0 "L4" V 6050 3400 50  0000 L CNN
 F 1 "2kH" V 6050 3200 50  0000 L CNN
 F 2 "Inductor_SMD:L_0805_2012Metric" V 5880 3350 50  0001 C CNN
@@
 $EndComp
 $Comp
-L Device:C_Small C21
+L Device:C_Small C31
 U 1 1 5C2B434A
 P 6550 3200
-F 0 "C21" H 6560 3270 50  0000 L CNN
+F 0 "C31" H 6560 3270 50  0000 L CNN
 F 1 "0.1uF" H 6560 3120 50  0000 L CNN
 F 2 "Capacitor_SMD:C_0805_2012Metric" H 6550 3200 50  0001 C CNN
@@
 $EndComp
 $Comp
-L Device:C_Small C22
+L Device:C_Small C32
 U 1 1 5C2B4351
 P 6850 3200
-F 0 "C22" H 6860 3270 50  0000 L CNN
+F 0 "C32" H 6860 3270 50  0000 L CNN
 F 1 "0.01uF" H 6860 3120 50  0000 L CNN
 F 2 "Capacitor_SMD:C_0805_2012Metric" H 6850 3200 50  0001 C CNN
@@
 $EndComp
 $Comp
-L utsvt-chips:ADM3055E U5
+L BPSMaster-rescue:ADM3055E-utsvt-chips U13
 U 1 1 5C2B4359
 P 4350 3600
-F 0 "U5" H 4100 4250 60  0000 C CNN
+F 0 "U13" H 4100 4250 60  0000 C CNN
 F 1 "ADM3055E" H 4550 3500 60  0000 C CNN
 F 2 "UTSVT_ICs:SOIC-20W_7.5x15.4mm_Pitch1.27mm" H 4350 3700 60  0001 C CNN
@@
 Text Notes 6550 2900 0    40   ~ 0
 Must be close\nto V_ISO_In
-$Comp
-L Connector:TestPoint TP6
-U 1 1 5C2B4371
-P 5100 2900
-F 0 "TP6" V 5200 3100 50  0000 L BNN
-F 1 "CAN_ISO_Vin" V 5100 3100 50  0000 L CNN
-F 2 "TestPoint:TestPoint_Keystone_5005-5009_Compact" H 5100 2900 50  0001 C CNN
-F 3 "" H 5100 2900 50  0001 C CNN
-	1    5100 2900
-	0    -1   -1   0
-$EndComp
-$Comp
-L Connector:TestPoint TP8
-U 1 1 5C2B4378
-P 6200 3700
-F 0 "TP8" V 6300 3900 50  0000 L BNN
-F 1 "CAN_ISO_GndOut" V 6200 3900 50  0000 L CNN
-F 2 "TestPoint:TestPoint_Keystone_5005-5009_Compact" H 6200 3700 50  0001 C CNN
-F 3 "" H 6200 3700 50  0001 C CNN
-	1    6200 3700
-	0    1    1    0
-$EndComp
-$Comp
-L Connector:TestPoint TP7
-U 1 1 5C2B437F
-P 6200 3550
-F 0 "TP7" V 6300 3750 50  0000 L BNN
-F 1 "CAN_ISO_GndIn" V 6200 3750 50  0000 L CNN
-F 2 "TestPoint:TestPoint_Keystone_5005-5009_Compact" H 6200 3550 50  0001 C CNN
-F 3 "" H 6200 3550 50  0001 C CNN
-	1    6200 3550
-	0    1    1    0
-$EndComp
-$Comp
-L Connector:TestPoint TP5
-U 1 1 5C2B4386
-P 5100 2750
-F 0 "TP5" V 5200 2950 50  0000 L BNN
-F 1 "CAN_ISO_Vout" V 5100 2950 50  0000 L CNN
-F 2 "TestPoint:TestPoint_Keystone_5005-5009_Compact" H 5100 2750 50  0001 C CNN
-F 3 "" H 5100 2750 50  0001 C CNN
-	1    5100 2750
-	0    -1   -1   0
-$EndComp
 NoConn ~ 3650 4100
 $Comp
-L power:PWR_FLAG #FLG03
+L power:PWR_FLAG #FLG04
 U 1 1 5C2B4394
 P 7300 3000
-F 0 "#FLG03" H 7300 3075 50  0001 C CNN
+F 0 "#FLG04" H 7300 3075 50  0001 C CNN
 F 1 "PWR_FLAG" H 7300 2900 30  0000 C CNN
 F 2 "" H 7300 3000 50  0001 C CNN
@@
 $EndComp
 $Comp
-L power:PWR_FLAG #FLG04
+L power:PWR_FLAG #FLG05
 U 1 1 5C2B439A
 P 7300 3200
-F 0 "#FLG04" H 7300 3275 50  0001 C CNN
+F 0 "#FLG05" H 7300 3275 50  0001 C CNN
 F 1 "PWR_FLAG" H 7200 3150 50  0001 L CNN
 F 2 "" H 7300 3200 50  0001 C CNN
@@
 $EndComp
 $Comp
-L utsvt-chips:CDSOT23-T24CAN U4
+L BPSMaster-rescue:CDSOT23-T24CAN-utsvt-chips U12
 U 1 1 5C2B43A0
 P 8100 2850
-F 0 "U4" H 8100 2700 60  0000 C CNN
+F 0 "U12" H 8100 2700 60  0000 C CNN
 F 1 "CDSOT23-T24CAN" H 8100 3000 60  0000 C CNN
 F 2 "Package_TO_SOT_SMD:SOT-23W" H 8100 2850 60  0001 C CNN
@@
 CAN Bus\nProtection
 $Comp
-L Connector:TestPoint TP9
+L Connector:TestPoint TP7
 U 1 1 5C2B43B6
 P 7300 3800
-F 0 "TP9" H 7300 4100 50  0000 C BNN
+F 0 "TP7" H 7300 4100 50  0000 C BNN
 F 1 "CAN_H" H 7300 4050 50  0000 C CNN
 F 2 "TestPoint:TestPoint_Keystone_5005-5009_Compact" H 7300 3800 50  0001 C CNN
@@
 $EndComp
 $Comp
-L Connector:TestPoint TP12
+L Connector:TestPoint TP8
 U 1 1 5C2B43BD
 P 7300 4000
-F 0 "TP12" H 7250 4200 50  0000 L BNN
+F 0 "TP8" H 7250 4200 50  0000 L BNN
 F 1 "CAN_L" H 7200 4300 50  0000 L CNN
 F 2 "TestPoint:TestPoint_Keystone_5005-5009_Compact" H 7300 4000 50  0001 C CNN
@@
 $EndComp
 $Comp
-L Device:R R4
+L Device:R R43
 U 1 1 5C2B43C4
 P 5550 4150
-F 0 "R4" V 5630 4150 50  0000 C CNN
+F 0 "R43" V 5630 4150 50  0000 C CNN
 F 1 "0" V 5550 4150 50  0000 C CNN
 F 2 "Resistor_SMD:R_0805_2012Metric" V 5480 4150 50  0001 C CNN
@@
 Wire Wire Line
 	5250 3150 5050 3150
-Wire Wire Line
-	5100 2900 5150 2900
 Wire Wire Line
 	5150 2900 5150 3050
@@
 Wire Wire Line
 	8200 3250 8200 3400
-Connection ~ 5150 2900
 Connection ~ 5250 3350
 Connection ~ 6150 3550
 Wire Wire Line
-	5100 2750 5250 2750
-Wire Wire Line
 	7300 3200 7300 3150
 Wire Wire Line
@@
 Wire Wire Line
 	5250 3050 5250 3150
-Wire Wire Line
-	5750 3350 5750 3700
-Wire Wire Line
-	6150 3550 6200 3550
-$Comp
-L power:GND #PWR042
+$Comp
+L power:GND #PWR071
 U 1 1 5C28BDDE
 P 2150 3550
-F 0 "#PWR042" H 2150 3300 50  0001 C CNN
+F 0 "#PWR071" H 2150 3300 50  0001 C CNN
 F 1 "GND" H 2300 3500 50  0000 C CNN
 F 2 "" H 2150 3550 50  0001 C CNN
@@
 	7300 3950 7550 3950
 Connection ~ 5750 3350
-Wire Wire Line
-	5250 3350 5750 3350
-Wire Wire Line
-	5750 3700 6200 3700
 Text Label 5050 3850 0    50   ~ 0
 CAN_H
@@
 Wire Wire Line
 	5250 3050 5750 3050
-Connection ~ 5250 3050
-Wire Wire Line
-	5150 2900 5250 2900
-Wire Wire Line
-	5250 2900 6150 2900
-Wire Wire Line
-	5250 2750 5250 3050
 Text Label 5050 4150 0    50   ~ 0
 RSlope
-Text HLabel 2050 3500 0    50   Input ~ 0
-GND
-Wire Wire Line
-	2050 3500 2150 3500
-Text HLabel 2400 3100 0    50   Input ~ 0
-+5V
-Wire Wire Line
-	2400 3100 2500 3100
-Text HLabel 2900 3200 0    50   Input ~ 0
-+3.3V
-Wire Wire Line
-	2900 3200 2950 3200
 Connection ~ 2950 3200
 Wire Wire Line
@@
 	2500 3000 2500 3100
 $Comp
-L power:+3.3V #PWR0133
+L power:+3.3V #PWR070
 U 1 1 5C4ABE05
 P 2950 3000
-F 0 "#PWR0133" H 2950 2850 50  0001 C CNN
+F 0 "#PWR070" H 2950 2850 50  0001 C CNN
 F 1 "+3.3V" H 2965 3173 50  0000 C CNN
 F 2 "" H 2950 3000 50  0001 C CNN
@@
 	2950 3000 2950 3200
 $Comp
-L power:+5V #PWR0132
+L power:+5V #PWR069
 U 1 1 5C4C2AB0
 P 2500 3000
-F 0 "#PWR0132" H 2500 2850 50  0001 C CNN
+F 0 "#PWR069" H 2500 2850 50  0001 C CNN
 F 1 "+5V" H 2515 3173 50  0000 C CNN
 F 2 "" H 2500 3000 50  0001 C CNN
@@
 Wire Wire Line
 	2950 3800 3650 3800
+Wire Wire Line
+	5150 2900 6150 2900
+Wire Wire Line
+	5250 3350 5750 3350
+Text Notes 7600 4250 0    50   ~ 0
+As long as total equals to 120 Ohms,\nthe two termination resistors can be any value
 $EndSCHEMATC
