File: BPS/Master/Contactor.sch (KiCad schematic (older format))
At the start: 20 parts, among them J6 ContactorConnector, Q1 VND5N07-E, Q2 NTR4003NT1G, U6 BAS70-04, U7 SI8261ABC-IS

Commit message: Adds master board v1.1.
Parts:
- C25: renamed from C27; value 1uF -> 1u
- C26: renamed from C28; value 10uF -> 10u
- C27: renamed from C29; value 0.1uF -> 0.1u
- C28: renamed from C30; value 1uF -> 1u
- U10: renamed from U6; symbol utsvt-bps:BAS70-04 -> BPSMaster-rescue:BAS70-04-utsvt-bps
- U11: renamed from U7; symbol utsvt-bps:SI8261ABC-IS -> BPSMaster-rescue:SI8261ABC-IS-utsvt-bps
- renumbered D2 to D10, D3 to D11, J6 to J7, R5 to R33, R6 to R34, R7 to R35, R8 to R36, R9 to R37, R10 to R38, R11 to R39, R12 to R40, TP13 to TP6
Connections:
- wire segments 77 -> 78
- no-connect marks 3 -> 2
