File: BPS/Master/Misc.sch (KiCad schematic (older format))
At the start: 34 parts, among them J11 FrontFans, J12 BackFans, J13 ErrorLightConnector, Q3 NTR4003NT1G, Q4 NTR4003NT1G, U16 SI8261ABC-IS

Commit message: Adds master board v1.1.
Parts:
- removed C48: 1uF, Capacitor_SMD:C_0805_2012Metric, symbol Device:C
- removed C49: 10uF, Capacitor_SMD:C_0805_2012Metric, symbol Device:C
- removed C50: 0.1uF, Capacitor_SMD:C_0805_2012Metric, symbol Device:C
- removed D4: 1N4148WS, Diode_SMD:D_SOD-323, symbol Device:D_ALT
- removed D5: Fault, LED_SMD:LED_0805_2012Metric, symbol Device:LED_ALT
- removed J13: ErrorLightConnector, UTSVT_Connectors:Molex_MicroFit3.0_1x2xP3.00mm_PolarizingPeg_Vertical, symbol Connector_Generic:Conn_01x02
- removed Q3, Q4: NTR4003NT1G, Package_TO_SOT_SMD:SOT-23, symbol Device:Q_NMOS_GSD
- removed R41: 1.6k, Resistor_SMD:R_0805_2012Metric, symbol Device:R
- removed R42: 470, Resistor_SMD:R_0805_2012Metric, symbol Device:R
- removed R43, R45: 0, Resistor_SMD:R_0805_2012Metric, symbol Device:R
- removed R44, R46: 10k, Resistor_SMD:R_0805_2012Metric, symbol Device:R
- removed TP14: StrobeLightGate_TP, TestPoint:TestPoint_Keystone_5005-5009_Compact, symbol Connector:TestPoint
- removed U16: SI8261ABC-IS, Package_SO:SOIC-8_3.9x4.9mm_P1.27mm, symbol utsvt-bps:SI8261ABC-IS
- renumbered D6 to D2, D7 to D3, D8 to D4, D9 to D5, D10 to D6, D11 to D7, D12 to D8, D13 to D9, J11 to J3, J12 to J4, R53 to R10, R54 to R11, R47 to R4, R48 to R5, R49 to R6, R50 to R7, R51 to R8, R52 to R9
Connections:
- net labels removed: +5V, FAULT
- wire segments 123 -> 64
- no-connect marks 3 -> 0
Other:
- note removed: "Error Light"
- note removed: "Please check footprint and symbol matches!\n1: G\n2: D\n3: S"
- note removed: "This page hods other miscellenious connections that are required:\n- Strobe/Error light indicator\n- Fan connectors"
- moved on the sheet: D2, D3, D4, D5, D6, D7, D8, D9, R10, R11, R4, R5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
