File: Dashboard/Dashboard/Dashboard.sch (KiCad schematic (older format))
At the start: 34 parts, among them J1 SWD, J10 Right Signal, J11 Brake Signal, J12 Headlight, J13 Vs-SPI3, J14 SPI3, J15 Vs-SPI1, J16 SPI1, J17 Vs-I2C3, J18 I2C3, J2 Logic Analyzer, J9 Left Signal, SW1 B3SL-1002P, U1 STM32F413RHTx, Y1 NX8045GB-8.000M-STD-CSJ-1

Commit message: Dashboard v2
Parts:
- removed J13: Vs-SPI3, Connector_PinHeader_2.54mm:PinHeader_1x03_P2.54mm_Vertical, symbol Connector_Generic:Conn_01x03
- added J5: Array Contactor 1, UTSVT_Connectors:Molex_MicroFit3.0_1x4xP3.00mm_PolarizingPeg_Vertical, symbol Connector_Generic:Conn_01x04
- added J6: Motor Contactor 1, UTSVT_Connectors:Molex_MicroFit3.0_1x4xP3.00mm_PolarizingPeg_Vertical, symbol Connector_Generic:Conn_01x04
- added J7: Array Contactor 2, UTSVT_Connectors:Molex_MicroFit3.0_1x4xP3.00mm_PolarizingPeg_Vertical, symbol Connector_Generic:Conn_01x04
- added J8: Motor Contactor 2, UTSVT_Connectors:Molex_MicroFit3.0_1x4xP3.00mm_PolarizingPeg_Vertical, symbol Connector_Generic:Conn_01x04
Connections:
- net +5V: now also J5.4 (Pin_4), J6.4 (Pin_4), J7.4 (Pin_4), J8.4 (Pin_4)
- net AC1_CHECK: now also J5.2 (Pin_2)
- net AC1_EN: now also J5.3 (Pin_3)
- net AC2_CHECK: now also J7.2 (Pin_2)
- net AC2_EN: now also J7.3 (Pin_3)
- net GND: now also J5.1 (Pin_1), J6.1 (Pin_1), J7.1 (Pin_1), J8.1 (Pin_1)
- net MC1_CHECK: now also J6.2 (Pin_2)
- net MC1_EN: now also J6.3 (Pin_3)
- net MC2_CHECK: now also J8.2 (Pin_2)
- net MC2_EN: now also J8.3 (Pin_3)
- net at J14.1 (Pin_1): now also J15.2 (Pin_2), J16.1 (Pin_1)
