File: BPS/Fuse/Fuse Board/Fuse Board.sch (KiCad schematic (older format))
At the start: 17 parts, among them J1 Conn_01x07, J2 Conn_01x06, J3 Conn_01x07, J4 Conn_01x06

Commit message: fuse board
Parts:
- F1, F10, F11, F12, F13, F2, F3, F4, F5, F6, F7, F8, F9: footprint Fuse:Fuse_0201_0603Metric -> UTSVT_BPS:MSF 250 Fuse
Changed lines of the file:
@@
 F 0 "F8" H 3450 2735 50  0000 C CNN
 F 1 "Fuse_Small" H 3450 2644 50  0000 C CNN
-F 2 "Fuse:Fuse_0201_0603Metric" H 3450 2550 50  0001 C CNN
+F 2 "UTSVT_BPS:MSF 250 Fuse" H 3450 2550 50  0001 C CNN
 F 3 "~" H 3450 2550 50  0001 C CNN
 	1    3450 2550
@@
 F 0 "F10" H 3450 3235 50  0000 C CNN
 F 1 "Fuse_Small" H 3450 3144 50  0000 C CNN
-F 2 "Fuse:Fuse_0201_0603Metric" H 3450 3050 50  0001 C CNN
+F 2 "UTSVT_BPS:MSF 250 Fuse" H 3450 3050 50  0001 C CNN
 F 3 "~" H 3450 3050 50  0001 C CNN
 	1    3450 3050
@@
 F 0 "F13" H 3450 3985 50  0000 C CNN
 F 1 "Fuse_Small" H 3450 3894 50  0000 C CNN
-F 2 "Fuse:Fuse_0201_0603Metric" H 3450 3800 50  0001 C CNN
+F 2 "UTSVT_BPS:MSF 250 Fuse" H 3450 3800 50  0001 C CNN
 F 3 "~" H 3450 3800 50  0001 C CNN
 	1    3450 3800
@@
 F 0 "F11" H 3450 3485 50  0000 C CNN
 F 1 "Fuse_Small" H 3450 3394 50  0000 C CNN
-F 2 "Fuse:Fuse_0201_0603Metric" H 3450 3300 50  0001 C CNN
+F 2 "UTSVT_BPS:MSF 250 Fuse" H 3450 3300 50  0001 C CNN
 F 3 "~" H 3450 3300 50  0001 C CNN
 	1    3450 3300
@@
 F 0 "F9" H 3450 2985 50  0000 C CNN
 F 1 "Fuse_Small" H 3450 2894 50  0000 C CNN
-F 2 "Fuse:Fuse_0201_0603Metric" H 3450 2800 50  0001 C CNN
+F 2 "UTSVT_BPS:MSF 250 Fuse" H 3450 2800 50  0001 C CNN
 F 3 "~" H 3450 2800 50  0001 C CNN
 	1    3450 2800
@@
 F 0 "F12" H 3450 3735 50  0000 C CNN
 F 1 "Fuse_Small" H 3450 3644 50  0000 C CNN
-F 2 "Fuse:Fuse_0201_0603Metric" H 3450 3550 50  0001 C CNN
+F 2 "UTSVT_BPS:MSF 250 Fuse" H 3450 3550 50  0001 C CNN
 F 3 "~" H 3450 3550 50  0001 C CNN
 	1    3450 3550
@@
 F 0 "F1" H 3250 4485 50  0000 C CNN
 F 1 "Fuse_Small" H 3250 4394 50  0000 C CNN
-F 2 "Fuse:Fuse_0201_0603Metric" H 3250 4300 50  0001 C CNN
+F 2 "UTSVT_BPS:MSF 250 Fuse" H 3250 4300 50  0001 C CNN
 F 3 "~" H 3250 4300 50  0001 C CNN
 	1    3250 4300
@@
 F 0 "F3" H 3250 4985 50  0000 C CNN
 F 1 "Fuse_Small" H 3250 4894 50  0000 C CNN
-F 2 "Fuse:Fuse_0201_0603Metric" H 3250 4800 50  0001 C CNN
+F 2 "UTSVT_BPS:MSF 250 Fuse" H 3250 4800 50  0001 C CNN
 F 3 "~" H 3250 4800 50  0001 C CNN
 	1    3250 4800
@@
 F 0 "F6" H 3250 5735 50  0000 C CNN
 F 1 "Fuse_Small" H 3250 5644 50  0000 C CNN
-F 2 "Fuse:Fuse_0201_0603Metric" H 3250 5550 50  0001 C CNN
+F 2 "UTSVT_BPS:MSF 250 Fuse" H 3250 5550 50  0001 C CNN
 F 3 "~" H 3250 5550 50  0001 C CNN
 	1    3250 5550
@@
 F 0 "F4" H 3250 5235 50  0000 C CNN
 F 1 "Fuse_Small" H 3250 5144 50  0000 C CNN
-F 2 "Fuse:Fuse_0201_0603Metric" H 3250 5050 50  0001 C CNN
+F 2 "UTSVT_BPS:MSF 250 Fuse" H 3250 5050 50  0001 C CNN
 F 3 "~" H 3250 5050 50  0001 C CNN
 	1    3250 5050
@@
 F 0 "F2" H 3250 4735 50  0000 C CNN
 F 1 "Fuse_Small" H 3250 4644 50  0000 C CNN
-F 2 "Fuse:Fuse_0201_0603Metric" H 3250 4550 50  0001 C CNN
+F 2 "UTSVT_BPS:MSF 250 Fuse" H 3250 4550 50  0001 C CNN
 F 3 "~" H 3250 4550 50  0001 C CNN
 	1    3250 4550
@@
 F 0 "F5" H 3250 5485 50  0000 C CNN
 F 1 "Fuse_Small" H 3250 5394 50  0000 C CNN
-F 2 "Fuse:Fuse_0201_0603Metric" H 3250 5300 50  0001 C CNN
+F 2 "UTSVT_BPS:MSF 250 Fuse" H 3250 5300 50  0001 C CNN
 F 3 "~" H 3250 5300 50  0001 C CNN
 	1    3250 5300
@@
 F 0 "F7" H 3250 5985 50  0000 C CNN
 F 1 "Fuse_Small" H 3250 5894 50  0000 C CNN
-F 2 "Fuse:Fuse_0201_0603Metric" H 3250 5800 50  0001 C CNN
+F 2 "UTSVT_BPS:MSF 250 Fuse" H 3250 5800 50  0001 C CNN
 F 3 "~" H 3250 5800 50  0001 C CNN
 	1    3250 5800
