File: BPS/Voltage/BPSVoltage.sch (KiCad schematic (older format))
At the start: 122 parts, among them J1 Conn1, J2 Conn2, J3 Conn_01x06, J4 Conn_01x07, J5 Conn_01x03, J6 Conn_01x05, J7 Conn_01x05, Q1 BSS308PE, Q10 BSS308PE, Q11 BSS308PE, Q12 BSS308PE, Q13 BSS308PE, Q2 BSS308PE, Q3 BSS308PE, Q4 BSS308PE, Q5 NSV1C201MZ4, Q6 BSS308PE, Q7 BSS308PE, Q8 BSS308PE, Q9 BSS308PE, U1 LTC6811-1, U2 HX1188FNL

Commit message: Relative addressing for schematic files
Parts:
- J1, J2: symbol BPSVoltage-rescue:CarPowerConnector-utsvt-connectors -> BPSVoltage-rescue:CarPowerConnector-utsvt-connectors-BPSVoltage-rescue
- U1: symbol BPSVoltage-rescue:LTC6811-1-utsvt-bps -> BPSVoltage-rescue:LTC6811-1-utsvt-bps-BPSVoltage-rescue
- U2: symbol BPSVoltage-rescue:HX1188FNL-utsvt-bps -> BPSVoltage-rescue:HX1188FNL-utsvt-bps-BPSVoltage-rescue
Changed lines of the file:
@@
 $EndDescr
 $Comp
-L BPSVoltage-rescue:LTC6811-1-utsvt-bps U1
+L BPSVoltage-rescue:LTC6811-1-utsvt-bps-BPSVoltage-rescue U1
 U 1 1 5C356477
 P 6400 2650
@@
 IMA
 $Comp
-L BPSVoltage-rescue:HX1188FNL-utsvt-bps U2
+L BPSVoltage-rescue:HX1188FNL-utsvt-bps-BPSVoltage-rescue U2
 U 1 1 5CAB08B5
 P 9700 5250
@@
 $EndComp
 $Comp
-L BPSVoltage-rescue:CarPowerConnector-utsvt-connectors J1
+L BPSVoltage-rescue:CarPowerConnector-utsvt-connectors-BPSVoltage-rescue J1
 U 1 1 5CAB16B3
 P 10750 5450
@@
 $EndComp
 $Comp
-L BPSVoltage-rescue:CarPowerConnector-utsvt-connectors J2
+L BPSVoltage-rescue:CarPowerConnector-utsvt-connectors-BPSVoltage-rescue J2
 U 1 1 5CADF981
 P 10750 5850

Commit message: Changed the connectors to stack
Parts:
- J1: footprint UTSVT_Connectors:Molex_MicroFit3.0_1x2xP3.00mm_PolarizingPeg_Vertical -> Connector_PinSocket_2.54mm:PinSocket_1x02_P2.54mm_Vertical_SMD_Pin1Right
- J2: footprint UTSVT_Connectors:Molex_MicroFit3.0_1x2xP3.00mm_PolarizingPeg_Vertical -> Connector_PinHeader_2.54mm:PinHeader_1x02_P2.54mm_Vertical_SMD_Pin1Right
Changed lines of the file:
@@
 F 0 "J1" H 10573 5508 60  0000 R CNN
 F 1 "Conn1" H 10573 5402 60  0000 R CNN
-F 2 "UTSVT_Connectors:Molex_MicroFit3.0_1x2xP3.00mm_PolarizingPeg_Vertical" H 10750 5450 60  0001 C CNN
+F 2 "Connector_PinSocket_2.54mm:PinSocket_1x02_P2.54mm_Vertical_SMD_Pin1Right" H 10750 5450 60  0001 C CNN
 F 3 "" H 10750 5450 60  0001 C CNN
 	1    10750 5450
@@
 F 0 "J2" H 10573 5908 60  0000 R CNN
 F 1 "Conn2" H 10573 5802 60  0000 R CNN
-F 2 "UTSVT_Connectors:Molex_MicroFit3.0_1x2xP3.00mm_PolarizingPeg_Vertical" H 10750 5850 60  0001 C CNN
+F 2 "Connector_PinHeader_2.54mm:PinHeader_1x02_P2.54mm_Vertical_SMD_Pin1Right" H 10750 5850 60  0001 C CNN
 F 3 "" H 10750 5850 60  0001 C CNN
 	1    10750 5850

Commit message: Edited comm pins of BPS voltage in case of stacking issues.
Parts:
- J5: footprint Connector_PinHeader_2.54mm:PinHeader_1x03_P2.54mm_Vertical -> Connector_PinHeader_2.00mm:PinHeader_1x03_P2.00mm_Vertical
Changed lines of the file:
@@
 F 0 "J5" H 9180 1142 50  0000 L CNN
 F 1 "Conn_01x03" H 9180 1051 50  0000 L CNN
-F 2 "Connector_PinHeader_2.54mm:PinHeader_1x03_P2.54mm_Vertical" H 9100 1100 50  0001 C CNN
+F 2 "Connector_PinHeader_2.00mm:PinHeader_1x03_P2.00mm_Vertical" H 9100 1100 50  0001 C CNN
 F 3 "~" H 9100 1100 50  0001 C CNN
 	1    9100 1100

Commit message: Redid the footprint for the IC, rerouted.
Parts:
- U1: footprint Package_SO:SSOP-48_7.5x15.9mm_P0.635mm -> UTSVT_ICs:SOIC-48
Changed lines of the file:
@@
 F 0 "U1" H 6400 2978 50  0000 C CNN
 F 1 "LTC6811-1" H 6400 2887 50  0000 C CNN
-F 2 "Package_SO:SSOP-48_7.5x15.9mm_P0.635mm" H 6400 2650 50  0001 C CNN
+F 2 "UTSVT_ICs:SOIC-48" H 6400 2650 50  0001 C CNN
 F 3 "" H 6400 2650 50  0001 C CNN
 	1    6400 2650

Commit message: Updated LTC6811 footprint.
Parts:
- added J8: Conn_01x02, UTSVT_Connectors:Molex_MicroFit3.0_1x2xP3.00mm_PolarizingPeg_Vertical, symbol Connector_Generic:Conn_01x02
Connections:
- wire segments 353 -> 359
Changed lines of the file:
@@
 $EndComp
 Wire Wire Line
-	10450 5350 10300 5350
-Wire Wire Line
-	10300 5550 10450 5550
+	10450 5350 10350 5350
+Wire Wire Line
+	10300 5550 10400 5550
 Wire Wire Line
 	10450 5750 10300 5750
@@
 Wire Notes Line
 	5850 7550 5850 6600
+$Comp
+L Connector_Generic:Conn_01x02 J8
+U 1 1 5C7F2BB2
+P 10700 4950
+F 0 "J8" H 10780 4942 50  0000 L CNN
+F 1 "Conn_01x02" H 10780 4851 50  0000 L CNN
+F 2 "UTSVT_Connectors:Molex_MicroFit3.0_1x2xP3.00mm_PolarizingPeg_Vertical" H 10700 4950 50  0001 C CNN
+F 3 "~" H 10700 4950 50  0001 C CNN
+	1    10700 4950
+	1    0    0    -1
+$EndComp
+Wire Wire Line
+	10400 5550 10400 5050
+Wire Wire Line
+	10400 5050 10500 5050
+Connection ~ 10400 5550
+Wire Wire Line
+	10400 5550 10450 5550
+Wire Wire Line
+	10350 5350 10350 4950
+Wire Wire Line
+	10350 4950 10500 4950
+Connection ~ 10350 5350
+Wire Wire Line
+	10350 5350 10300 5350
 $EndSCHEMATC

Commit message: footprint error fixed in voltage board. Created new gerber files.
Parts:
- U1: footprint UTSVT_ICs:SOIC-48 -> UTSVT_BPS:LTC6811HG-1-PBF
Changed lines of the file:
@@
 F 0 "U1" H 6400 2978 50  0000 C CNN
 F 1 "LTC6811-1" H 6400 2887 50  0000 C CNN
-F 2 "UTSVT_ICs:SOIC-48" H 6400 2650 50  0001 C CNN
+F 2 "UTSVT_BPS:LTC6811HG-1-PBF" H 6400 2650 50  0001 C CNN
 F 3 "" H 6400 2650 50  0001 C CNN
 	1    6400 2650

Commit message: Edited temmperature board to have reset pin to high.
Parts:
- C10, C8, C9: value 10u -> 1u
Changed lines of the file:
@@
 P 8300 3500
 F 0 "C8" H 8415 3546 50  0000 L CNN
-F 1 "10u" H 8415 3455 50  0000 L CNN
+F 1 "1u" H 8415 3455 50  0000 L CNN
 F 2 "Capacitor_SMD:C_0805_2012Metric" H 8338 3350 50  0001 C CNN
 F 3 "~" H 8300 3500 50  0001 C CNN
@@
 P 8650 3500
 F 0 "C9" H 8765 3546 50  0000 L CNN
-F 1 "10u" H 8765 3455 50  0000 L CNN
+F 1 "1u" H 8765 3455 50  0000 L CNN
 F 2 "Capacitor_SMD:C_0805_2012Metric" H 8688 3350 50  0001 C CNN
 F 3 "~" H 8650 3500 50  0001 C CNN
@@
 P 9000 3500
 F 0 "C10" H 9115 3546 50  0000 L CNN
-F 1 "10u" H 9115 3455 50  0000 L CNN
+F 1 "1u" H 9115 3455 50  0000 L CNN
 F 2 "Capacitor_SMD:C_0805_2012Metric" H 9038 3350 50  0001 C CNN
 F 3 "~" H 9000 3500 50  0001 C CNN
