File: BPS/Master-Nucleo/PowerDist.sch (KiCad schematic (older format))
At the start: 15 parts, among them J4 CarPowerConnector, U2 RI3-1205S, U3 NCP1117-3.3_SOT223

Commit message: Adds Nucleo version of master board.
Parts:
- removed C17, C18: 10uF, Capacitor_SMD:C_0805_2012Metric, symbol Device:C
- removed TP4: +3.3V_TP, TestPoint:TestPoint_Keystone_5005-5009_Compact, symbol Connector:TestPoint
- removed U3: NCP1117-3.3_SOT223, Package_TO_SOT_SMD:SOT-223-3_TabPin2, symbol Regulator_Linear:LD1117S33TR_SOT223
- renumbered C15 to C5, C16 to C6, D1 to D3, J4 to J2, R1 to R9, TP1 to TP2, TP2 to TP3, TP15 to TP4, TP3 to TP5, U2 to U4
Connections:
- net labels removed: +3.3V
- wire segments 64 -> 49
Changed lines of the file:
@@
 EESchema Schematic File Version 4
-LIBS:BPSMaster-cache
 EELAYER 29 0
 EELAYER END
 $Descr A4 11693 8268
 encoding utf-8
-Sheet 2 7
+Sheet 3 7
 Title ""
 Date ""
@@
 $EndDescr
 $Comp
-L utsvt-connectors:CarPowerConnector J4
+L utsvt-connectors:CarPowerConnector J2
 U 1 1 5C35F236
 P 2100 3400
-F 0 "J4" H 2150 3750 60  0000 C CNN
+F 0 "J2" H 2150 3750 60  0000 C CNN
 F 1 "CarPowerConnector" H 1800 3650 60  0000 C CNN
 F 2 "UTSVT_Connectors:Molex_MicroFit3.0_1x2xP3.00mm_PolarizingPeg_Vertical" H 2100 3400 60  0001 C CNN
@@
 	2450 3500 2450 3600
 $Comp
-L power:+12V #PWR034
+L power:+12V #PWR0113
 U 1 1 5C35F2D2
 P 2450 3150
-F 0 "#PWR034" H 2450 3000 50  0001 C CNN
+F 0 "#PWR0113" H 2450 3000 50  0001 C CNN
 F 1 "+12V" H 2465 3323 50  0000 C CNN
 F 2 "" H 2450 3150 50  0001 C CNN
@@
 	2450 3600 2450 3650
 $Comp
-L Device:C C16
+L Device:C C6
 U 1 1 5C35F7E4
 P 2700 3400
-F 0 "C16" H 2818 3446 50  0000 L CNN
+F 0 "C6" H 2818 3446 50  0000 L CNN
 F 1 "4.7uF" H 2818 3355 50  0000 L CNN
 F 2 "Capacitor_SMD:C_0805_2012Metric" H 2738 3250 50  0001 C CNN
@@
 Connection ~ 5200 3600
 $Comp
-L Device:C C15
+L Device:C C5
 U 1 1 5C3626E7
 P 4550 2850
-F 0 "C15" H 4668 2896 50  0000 L CNN
+F 0 "C5" H 4668 2896 50  0000 L CNN
 F 1 "470pF" H 4668 2805 50  0000 L CNN
 F 2 "Capacitor_SMD:C_2220_5650Metric" H 4588 2700 50  0001 C CNN
@@
 +5V
 $Comp
-L power:+5V #PWR035
+L power:+5V #PWR0114
 U 1 1 5C376123
 P 5200 3150
-F 0 "#PWR035" H 5200 3000 50  0001 C CNN
+F 0 "#PWR0114" H 5200 3000 50  0001 C CNN
 F 1 "+5V" H 5215 3323 50  0000 C CNN
 F 2 "" H 5200 3150 50  0001 C CNN
@@
 $EndComp
 $Comp
-L Connector:TestPoint TP1
+L Connector:TestPoint TP2
 U 1 1 5C37D606
 P 2700 3150
-F 0 "TP1" H 2700 3500 50  0000 L CNN
+F 0 "TP2" H 2700 3500 50  0000 L CNN
 F 1 "+12V_TP" H 2700 3400 50  0000 L CNN
 F 2 "TestPoint:TestPoint_Keystone_5005-5009_Compact" H 2900 3150 50  0001 C CNN
@@
 	2700 3150 2700 3200
 $Comp
-L Connector:TestPoint TP2
+L Connector:TestPoint TP3
 U 1 1 5C37E6A3
 P 5500 3150
-F 0 "TP2" H 5558 3270 50  0000 L CNN
+F 0 "TP3" H 5558 3270 50  0000 L CNN
 F 1 "+5V_TP" H 5558 3179 50  0000 L CNN
 F 2 "TestPoint:TestPoint_Keystone_5005-5009_Compact" H 5700 3150 50  0001 C CNN
@@
 	5500 3150 5500 3200
 $Comp
-L Connector:TestPoint TP3
+L Connector:TestPoint TP5
 U 1 1 5C37F6B1
 P 5500 3700
-F 0 "TP3" H 5442 3727 50  0000 R CNN
+F 0 "TP5" H 5442 3727 50  0000 R CNN
 F 1 "GND_TP" H 5442 3818 50  0000 R CNN
 F 2 "TestPoint:TestPoint_Keystone_5005-5009_Compact" H 5700 3700 50  0001 C CNN
@@
 	5500 3700 5500 3600
 $Comp
-L power:GND #PWR038
+L power:GND #PWR0115
 U 1 1 5C58D746
 P 6350 3800
-F 0 "#PWR038" H 6350 3550 50  0001 C CNN
+F 0 "#PWR0115" H 6350 3550 50  0001 C CNN
 F 1 "GND" H 6355 3627 50  0000 C CNN
 F 2 "" H 6350 3800 50  0001 C CNN
@@
 $EndComp
 $Comp
-L Device:LED_ALT D1
+L Device:LED_ALT D3
 U 1 1 5C58D83E
 P 6350 3600
-F 0 "D1" V 6388 3482 50  0000 R CNN
+F 0 "D3" V 6388 3482 50  0000 R CNN
 F 1 "PowerOn" V 6297 3482 50  0000 R CNN
 F 2 "LED_SMD:LED_0805_2012Metric" H 6350 3600 50  0001 C CNN
@@
 $EndComp
 $Comp
-L Device:R R1
+L Device:R R9
 U 1 1 5C58D993
 P 6350 3250
-F 0 "R1" H 6420 3296 50  0000 L CNN
+F 0 "R9" H 6420 3296 50  0000 L CNN
 F 1 "1.5k" H 6420 3205 50  0000 L CNN
 F 2 "Resistor_SMD:R_0805_2012Metric" V 6280 3250 50  0001 C CNN
@@
 	6350 3450 6350 3400
 $Comp
-L power:+5V #PWR033
+L power:+5V #PWR0116
 U 1 1 5C58FEF6
 P 6350 3050
-F 0 "#PWR033" H 6350 2900 50  0001 C CNN
+F 0 "#PWR0116" H 6350 2900 50  0001 C CNN
 F 1 "+5V" H 6365 3223 50  0000 C CNN
 F 2 "" H 6350 3050 50  0001 C CNN
@@
 	6350 3050 6350 3100
 $Comp
-L power:GND #PWR037
+L power:GND #PWR0117
 U 1 1 5C3F3B1F
 P 5200 3700
-F 0 "#PWR037" H 5200 3450 50  0001 C CNN
+F 0 "#PWR0117" H 5200 3450 50  0001 C CNN
 F 1 "GND" H 5205 3527 50  0000 C CNN
 F 2 "" H 5200 3700 50  0001 C CNN
@@
 $EndComp
 $Comp
-L power:GNDPWR #PWR036
+L power:GNDPWR #PWR0118
 U 1 1 5C3F7204
 P 2450 3650
-F 0 "#PWR036" H 2450 3450 50  0001 C CNN
+F 0 "#PWR0118" H 2450 3450 50  0001 C CNN
 F 1 "GNDPWR" H 2454 3496 50  0000 C CNN
 F 2 "" H 2450 3600 50  0001 C CNN
@@
 $EndComp
 $Comp
-L power:+5V #PWR039
-U 1 1 5C702374
-P 4300 4400
-F 0 "#PWR039" H 4300 4250 50  0001 C CNN
-F 1 "+5V" H 4315 4573 50  0000 C CNN
-F 2 "" H 4300 4400 50  0001 C CNN
-F 3 "" H 4300 4400 50  0001 C CNN
-	1    4300 4400
-	1    0    0    -1
-$EndComp
-$Comp
-L Regulator_Linear:LD1117S33TR_SOT223 U3
-U 1 1 5C70247C
-P 4800 4500
-F 0 "U3" H 4800 4742 50  0000 C CNN
-F 1 "NCP1117-3.3_SOT223" H 4800 4651 50  0000 C CNN
-F 2 "Package_TO_SOT_SMD:SOT-223-3_TabPin2" H 4800 4700 50  0001 C CNN
-F 3 "http://www.onsemi.com/pub_link/Collateral/NCP1117-D.PDF" H 4900 4250 50  0001 C CNN
-	1    4800 4500
-	1    0    0    -1
-$EndComp
-$Comp
-L Device:C C17
-U 1 1 5C702937
-P 4300 4700
-F 0 "C17" H 4415 4746 50  0000 L CNN
-F 1 "10uF" H 4415 4655 50  0000 L CNN
-F 2 "Capacitor_SMD:C_0805_2012Metric" H 4338 4550 50  0001 C CNN
-F 3 "~" H 4300 4700 50  0001 C CNN
-	1    4300 4700
-	1    0    0    -1
-$EndComp
-$Comp
-L Device:C C18
-U 1 1 5C7029C7
-P 5300 4700
-F 0 "C18" H 5415 4746 50  0000 L CNN
-F 1 "10uF" H 5415 4655 50  0000 L CNN
-F 2 "Capacitor_SMD:C_0805_2012Metric" H 5338 4550 50  0001 C CNN
-F 3 "~" H 5300 4700 50  0001 C CNN
-	1    5300 4700
-	1    0    0    -1
-$EndComp
-Wire Wire Line
-	4500 4500 4300 4500
-Wire Wire Line
-	4300 4500 4300 4550
-Wire Wire Line
-	5100 4500 5300 4500
-Wire Wire Line
-	5300 4500 5300 4550
-$Comp
-L power:GND #PWR041
-U 1 1 5C703BF4
-P 4800 4950
-F 0 "#PWR041" H 4800 4700 50  0001 C CNN
-F 1 "GND" H 4805 4777 50  0000 C CNN
-F 2 "" H 4800 4950 50  0001 C CNN
-F 3 "" H 4800 4950 50  0001 C CNN
-	1    4800 4950
-	1    0    0    -1
-$EndComp
-Wire Wire Line
-	4300 4850 4300 4900
-Wire Wire Line
-	4300 4900 4800 4900
-Wire Wire Line
-	5300 4900 5300 4850
-Wire Wire Line
-	4800 4800 4800 4900
-Connection ~ 4800 4900
-Wire Wire Line
-	4800 4900 5300 4900
-Wire Wire Line
-	4800 4900 4800 4950
-Wire Wire Line
-	4300 4400 4300 4500
-Connection ~ 4300 4500
-$Comp
-L power:+3.3V #PWR040
-U 1 1 5C7065C8
-P 5300 4400
-F 0 "#PWR040" H 5300 4250 50  0001 C CNN
-F 1 "+3.3V" H 5315 4573 50  0000 C CNN
-F 2 "" H 5300 4400 50  0001 C CNN
-F 3 "" H 5300 4400 50  0001 C CNN
-	1    5300 4400
-	1    0    0    -1
-$EndComp
-Wire Wire Line
-	5300 4400 5300 4500
-Connection ~ 5300 4500
-Text HLabel 5700 4500 2    50   Input ~ 0
-+3.3V
-Wire Wire Line
-	5700 4500 5500 4500
-$Comp
-L Connector:TestPoint TP4
-U 1 1 5C708412
-P 5500 4450
-F 0 "TP4" H 5558 4570 50  0000 L CNN
-F 1 "+3.3V_TP" H 5550 4650 50  0000 L CNN
-F 2 "TestPoint:TestPoint_Keystone_5005-5009_Compact" H 5700 4450 50  0001 C CNN
-F 3 "~" H 5700 4450 50  0001 C CNN
-	1    5500 4450
-	1    0    0    -1
-$EndComp
-Wire Wire Line
-	5500 4450 5500 4500
-Connection ~ 5500 4500
-Wire Wire Line
-	5500 4500 5300 4500
-$Comp
-L power:PWR_FLAG #FLG02
+L power:PWR_FLAG #FLG0101
 U 1 1 5CC7C643
 P 4000 2750
-F 0 "#FLG02" H 4000 2825 50  0001 C CNN
+F 0 "#FLG0101" H 4000 2825 50  0001 C CNN
 F 1 "PWR_FLAG" H 4000 2924 50  0000 C CNN
 F 2 "" H 4000 2750 50  0001 C CNN
@@
 	4000 2750 4000 2850
 $Comp
-L utsvt-power-regulators:RI3-1205S U2
+L utsvt-power-regulators:RI3-1205S U4
 U 1 1 5C38C4FE
 P 4550 3200
-F 0 "U2" H 4550 3365 50  0000 C CNN
+F 0 "U4" H 4550 3365 50  0000 C CNN
 F 1 "RI3-1205S" H 4550 3274 50  0000 C CNN
 F 2 "UTSVT_ICs:RI3_DC_Converter" H 4550 3200 50  0001 C CNN
@@
 Connection ~ 5100 3200
 $Comp
-L Connector:TestPoint TP15
+L Connector:TestPoint TP4
 U 1 1 5C82CEA3
 P 2700 3650
-F 0 "TP15" H 2642 3677 50  0000 R CNN
+F 0 "TP4" H 2642 3677 50  0000 R CNN
 F 1 "GNDPWR_TP" H 2642 3768 50  0000 R CNN
 F 2 "TestPoint:TestPoint_Keystone_5005-5009_Compact" H 2900 3650 50  0001 C CNN
