File: BPS/Display/PowerDist.sch (KiCad schematic (older format))
At the start: 15 parts, among them J4 CarPowerConnector, U2 RI3-1205S, U3 NCP1117-3.3_SOT223

Commit message: Adds display board
Parts:
- removed C15: 470pF, Capacitor_SMD:C_2220_5650Metric, symbol Device:C
- removed C17, C18: 10uF, Capacitor_SMD:C_0805_2012Metric, symbol Device:C
- removed L1: 10uH, UTSVT_BPS:SRF0905A, symbol utsvt-bps:SRF0905-100Y
- removed TP4: +3.3V_TP, TestPoint:TestPoint_Keystone_5005-5009_Compact, symbol Connector:TestPoint
- removed U2: RI3-1205S, UTSVT_ICs:RI3_DC_Converter, symbol utsvt-power-regulators:RI3-1205S
- removed U3: NCP1117-3.3_SOT223, Package_TO_SOT_SMD:SOT-223-3_TabPin2, symbol Regulator_Linear:LD1117S33TR_SOT223
- added C23: 4.7u, Capacitor_SMD:C_0805_2012Metric, symbol Device:C
- added C24, C25: 10u, Capacitor_SMD:C_0805_2012Metric, symbol Device:C
- added L3: 6.8u, Inductor_SMD:L_Taiyo-Yuden_MD-4040, symbol Device:L
- added U6: PDS1-S12-S5, UTSVT_ICs:PDSx-S, symbol utsvt-power-regulators:PDS1-Sx-Sx
- added U7: NCP1117-3.3_SOT223, Package_TO_SOT_SMD:SOT-223-3_TabPin2, symbol Regulator_Linear:NCP1117-3.3_SOT223
- C22: renamed from C16; value 4.7uF -> 4.7u
- J5: renamed from J4; footprint UTSVT_Connectors:Molex_MicroFit3.0_1x2xP3.00mm_PolarizingPeg_Vertical -> Connector_Molex:Molex_Micro-Fit_3.0_43650-0200_1x02_P3.00mm_Horizontal
- TP3: renamed from TP2; value +5V_TP -> +3.3V_TP
- renumbered R1 to R7, TP1 to TP4, TP15 to TP5, TP3 to TP6
Connections:
- wire segments 64 -> 52
Other:
- moved on the sheet: TP3, TP6
