File: ContactorDriver/_autosave-ContactorDriver.sch (KiCad schematic (older format))
At the start: 36 parts, among them J1 PowerConn, J2 DashboardConn, J3 DashboardConn, J4 ContactorConn, J5 PrechargeConn, Q1 NTR4003NT1G, Q2 NTR4003NT1G, Q3 CSD18511KTT, Q4 CSD18511KTT

Commit message: Adds resistor mount. Need to add pheonix connector.
Parts:
- added H?: MountingHole_Pad, symbol Mechanical:MountingHole_Pad
Other:
- moved on the sheet: D1, R1
Changed lines of the file:
@@
 L Device:R_Small R1
 U 1 1 5E3A03D5
-P 3050 1600
-F 0 "R1" H 3150 1700 50  0000 C CNN
-F 1 "10k" H 3155 1600 50  0000 C CNN
-F 2 "Resistor_SMD:R_0805_2012Metric_Pad1.15x1.40mm_HandSolder" H 3050 1600 50  0001 C CNN
-F 3 "~" H 3050 1600 50  0001 C CNN
-	1    3050 1600
+P 2600 1450
+F 0 "R1" H 2700 1550 50  0000 C CNN
+F 1 "10k" H 2705 1450 50  0000 C CNN
+F 2 "Resistor_SMD:R_0805_2012Metric_Pad1.15x1.40mm_HandSolder" H 2600 1450 50  0001 C CNN
+F 3 "~" H 2600 1450 50  0001 C CNN
+	1    2600 1450
 	1    0    0    1
 $EndComp
@@
 L Device:LED_Small D1
 U 1 1 5E3A03DC
-P 3050 1900
-F 0 "D1" V 3096 1832 50  0000 R CNN
-F 1 "Green" V 3005 1832 50  0000 R CNN
-F 2 "LED_SMD:LED_0805_2012Metric_Pad1.15x1.40mm_HandSolder" V 3050 1900 50  0001 C CNN
-F 3 "~" V 3050 1900 50  0001 C CNN
-	1    3050 1900
+P 2600 1750
+F 0 "D1" V 2646 1682 50  0000 R CNN
+F 1 "Green" V 2555 1682 50  0000 R CNN
+F 2 "LED_SMD:LED_0805_2012Metric_Pad1.15x1.40mm_HandSolder" V 2600 1750 50  0001 C CNN
+F 3 "~" V 2600 1750 50  0001 C CNN
+	1    2600 1750
 	0    1    -1   0
 $EndComp
 Wire Wire Line
-	3050 1800 3050 1700
+	2600 1650 2600 1550
 $Comp
 L power:GND #PWR04
 U 1 1 5E3A4D78
-P 3050 2100
-F 0 "#PWR04" H 3050 1850 50  0001 C CNN
-F 1 "GND" H 3055 1927 50  0000 C CNN
-F 2 "" H 3050 2100 50  0001 C CNN
-F 3 "" H 3050 2100 50  0001 C CNN
-	1    3050 2100
+P 2600 1950
+F 0 "#PWR04" H 2600 1700 50  0001 C CNN
+F 1 "GND" H 2605 1777 50  0000 C CNN
+F 2 "" H 2600 1950 50  0001 C CNN
+F 3 "" H 2600 1950 50  0001 C CNN
+	1    2600 1950
 	1    0    0    -1
 $EndComp
 Wire Wire Line
-	3050 2100 3050 2000
+	2600 1950 2600 1850
 $Comp
 L power:+12V #PWR03
 U 1 1 5E3AC7F0
-P 3050 1400
-F 0 "#PWR03" H 3050 1250 50  0001 C CNN
-F 1 "+12V" H 3065 1573 50  0000 C CNN
-F 2 "" H 3050 1400 50  0001 C CNN
-F 3 "" H 3050 1400 50  0001 C CNN
-	1    3050 1400
+P 2600 1250
+F 0 "#PWR03" H 2600 1100 50  0001 C CNN
+F 1 "+12V" H 2615 1423 50  0000 C CNN
+F 2 "" H 2600 1250 50  0001 C CNN
+F 3 "" H 2600 1250 50  0001 C CNN
+	1    2600 1250
 	1    0    0    -1
 $EndComp
 Wire Wire Line
-	3050 1400 3050 1500
+	2600 1250 2600 1350
 $Comp
 L Mechanical:MountingHole H2
@@
 	1    0    0    -1
 $EndComp
+$Comp
+L Mechanical:MountingHole_Pad H?
+U 1 1 5E2EBBBD
+P 9400 3600
+F 0 "H?" H 9500 3649 50  0000 L CNN
+F 1 "MountingHole_Pad" H 9500 3558 50  0000 L CNN
+F 2 "" H 9400 3600 50  0001 C CNN
+F 3 "~" H 9400 3600 50  0001 C CNN
+	1    9400 3600
+	1    0    0    -1
+$EndComp
