File: Array/RTD Temp Board/RTDTemp.kicad_pcb (KiCad board)
At the start: 2 copper layers, 114.5 x 60 mm, 94 parts, among them J1 Conn_01x02, J10 Conn_01x02, J11 Conn_01x02, J2 Conn_01x02, J3 Conn_01x02, J4 CAN_In, J5 CAN_Out, J6 Conn_01x02, J7 Conn_01x02, J8 Conn_01x02, J9 Conn_01x02, U1 INA21x, U10 INA21x, U11 INA21x, U12 INA21x, U2 Nucleo_L432KC, U3 PDS1-Sx-Sx, U4 INA21x, U5 ADM3055E, U6 INA21x, U7 CDSOT23-T24CAN, U8 INA21x, U9 INA21x

Commit message: Editing Array and Starting Telemetry board
Parts:
- added RTD0: TestPoint, TestPoint:TestPoint_Keystone_5005-5009_Compact, F.Cu at (195.1, 75.2)
- added TP1: TestPoint, TestPoint:TestPoint_Keystone_5005-5009_Compact, F.Cu at (129.1, 75.2)
- added TP2: TestPoint, TestPoint:TestPoint_Keystone_5005-5009_Compact, F.Cu at (118.0, 75.2)
- added TP3: TestPoint, TestPoint:TestPoint_Keystone_5005-5009_Compact, F.Cu at (151.1, 75.2)
- added TP4: TestPoint, TestPoint:TestPoint_Keystone_5005-5009_Compact, F.Cu at (140.1, 75.2)
- added TP6: TestPoint, TestPoint:TestPoint_Keystone_5005-5009_Compact, F.Cu at (184.1, 75.2)
- added TP7: TestPoint, TestPoint:TestPoint_Keystone_5005-5009_Compact, F.Cu at (173.1, 75.2)
- added TP8: TestPoint, TestPoint:TestPoint_Keystone_5005-5009_Compact, F.Cu at (162.1, 75.2)
- moved LED7 6.34 mm to (113.6, 89.2), turned to 0 degrees
- moved LED3 2.24 mm to (113.5, 92.2)
Routing:
- net GND: track 191.4 -> 171.8 mm
- net Net-(LED7-Pad2): track 3.73 -> 9.81 mm
- net /RTD4: track 10.1 -> 15.2 mm
- net /RTD0: track 39.5 -> 44.3 mm
- net /RTD2: track 22.6 -> 27.4 mm
- net /RTD1: track 31.0 -> 35.9 mm
- net /RTD3: track 14.4 -> 19.2 mm
- net /RTD6: track 23.8 -> 27.7 mm
- net /RTD7: track 32.2 -> 36.1 mm
- net /RTD5: track 15.3 -> 19.2 mm
Other:
- board text added: "RTD1"
- board text added: "RTD2"
- board text added: "RTD3"
- board text added: "RTD4"
- board text added: "RTD5"
- board text added: "RTD6"
- board text added: "RTD7"
