File: Array/RTD Temp Board/RTDTemp.sch (KiCad schematic (older format))
At the start: 92 parts, among them J1 Conn_01x02, J10 Conn_01x02, J11 Conn_01x02, J2 Conn_01x02, J3 Conn_01x02, J4 CAN_In, J5 CAN_Out, J6 Conn_01x02, J7 Conn_01x02, J8 Conn_01x02, J9 Conn_01x02, U1 INA21x, U10 INA21x, U11 INA21x, U12 INA21x, U2 Nucleo_L432KC, U3 PDS1-Sx-Sx, U4 INA21x, U5 ADM3055E, U6 INA21x, U7 CDSOT23-T24CAN, U8 INA21x, U9 INA21x

Commit message: Editing Array and Starting Telemetry board
Parts:
- added TP1, TP2, TP3, TP4, TP5, TP6, TP7, TP8: TestPoint, TestPoint:TestPoint_Keystone_5005-5009_Compact, symbol Connector:TestPoint
- C10, C11, C12, C13, C14, C15, C16, C9: symbol MPPT-rescue:C_Small -> RTDTemp-rescue:C_Small-MPPT-rescue
- J4, J5: symbol MPPT-rescue:CANConnector -> RTDTemp-rescue:CANConnector-MPPT-rescue
- JP1: symbol MPPT-rescue:Jumper_NO_Small -> RTDTemp-rescue:Jumper_NO_Small-MPPT-rescue
- L2, L3: symbol MPPT-rescue:Ferrite_Bead_Small -> RTDTemp-rescue:Ferrite_Bead_Small-MPPT-rescue
- LED3, LED7, LED8, LED9: symbol MPPT-rescue:LED_ALT -> RTDTemp-rescue:LED_ALT-MPPT-rescue
- R10, R25, R9: symbol MPPT-rescue:R -> RTDTemp-rescue:R-MPPT-rescue
- R14, R20, R21, R22: symbol MPPT-rescue:R_Small -> RTDTemp-rescue:R_Small-MPPT-rescue
- TP13, TP14, TP15, TP16, TP19, TP20, TP21, TP22, TP26: symbol MPPT-rescue:TEST -> RTDTemp-rescue:TEST-MPPT-rescue
- U1, U10, U11, U12, U4, U6, U8, U9: symbol MPPT-rescue:INA21x -> RTDTemp-rescue:INA21x-MPPT-rescue
- U2: symbol MPPT-rescue:Nucleo_L432KC -> RTDTemp-rescue:Nucleo_L432KC-MPPT-rescue
- U5: symbol MPPT-rescue:ADM3055E -> RTDTemp-rescue:ADM3055E-MPPT-rescue
- U7: symbol MPPT-rescue:CDSOT23-T24CAN -> RTDTemp-rescue:CDSOT23-T24CAN-MPPT-rescue
Connections:
- net RTD0: now also TP5.1
- net RTD1: now also TP6.1
- net RTD2: now also TP7.1
- net RTD3: now also TP8.1
- net RTD4: now also TP3.1
- net RTD5: now also TP4.1
- net RTD6: now also TP1.1
- net RTD7: now also TP2.1
