File: BPS/Leader/EEPROM.sch (KiCad schematic (older format))
At the start: 4 parts, among them U4 M24128

Commit message: Leader board (#42)
* Creates fan brd interface schematics and updates symbols/footprints related to the leader board

* Finishes schematics for bps leader board

* Renames bps master to bps leader:

* Places most components of leader board in their respective locations with nothing traced

* Adds power planes

* Everything traced in leader board except for power circuitry

* Traces power components

* Finished leader board

* Simplifies dc-dc converter schematics

* Updates leader board, need to add comments

* Finishes new power circuitry tracing

* Adds version number to leader_board and creates schematics pdf

* Edits diode V2F22HM footprint to not have a copper cutout

* Adds copper cutout to transformer for isospi because ltc6820 datasheet recommended it

* Changes LTC6820 POL and PHA pins to +5V due to VIH and VIL parameters in datasheet

* Checks and make sure everything passes DRC

* Updates V2F22HM footprint to include polarity indicator on silkscreen

* Adds documents/pdfs to leader board

* Deletes errenous pdf

* Checks ERC/DRC one more time

* Updates LTC6820 symbol

* Removes previous current board interface hierachy sheet

* These twwo files were combined into SensorBrdInterface.sch
Parts:
- removed U4: M24128, UTSVT_BPS:M24128-BRMN6P, symbol BPSMaster-rescue:M24128-utsvt-bps
- added U4: M24128, Package_SO:SOIC-8_3.9x4.9mm_P1.27mm, symbol utsvt-bps:M24128
- C15: renamed from C16; value 0.1uF -> 0.1u
Changed lines of the file:
@@
 $Descr A4 11693 8268
 encoding utf-8
-Sheet 3 10
+Sheet 3 11
 Title ""
 Date ""
@@
 SCL
 $Comp
-L BPSMaster-rescue:M24128-utsvt-bps U4
-U 1 1 5C3511BE
-P 4250 2800
-F 0 "U4" H 4250 2965 50  0000 C CNN
-F 1 "M24128" H 4250 2874 50  0000 C CNN
-F 2 "UTSVT_BPS:M24128-BRMN6P" H 4250 2800 50  0001 C CNN
-F 3 "" H 4250 2800 50  0001 C CNN
-	1    4250 2800
-	-1   0    0    -1
-$EndComp
-$Comp
-L Device:C C16
+L Device:C C15
 U 1 1 5C35143C
 P 3200 2800
-F 0 "C16" H 3315 2846 50  0000 L CNN
-F 1 "0.1uF" H 3315 2755 50  0000 L CNN
+F 0 "C15" H 3315 2846 50  0000 L CNN
+F 1 "0.1u" H 3315 2755 50  0000 L CNN
 F 2 "Capacitor_SMD:C_0805_2012Metric" H 3238 2650 50  0001 C CNN
 F 3 "~" H 3200 2800 50  0001 C CNN
@@
 $EndComp
 $Comp
-L power:GND #PWR027
+L power:GND #PWR032
 U 1 1 5C3514DC
 P 4850 3300
-F 0 "#PWR027" H 4850 3050 50  0001 C CNN
+F 0 "#PWR032" H 4850 3050 50  0001 C CNN
 F 1 "GND" H 4855 3127 50  0000 C CNN
 F 2 "" H 4850 3300 50  0001 C CNN
@@
 Connection ~ 4850 3200
 $Comp
-L power:GND #PWR026
+L power:GND #PWR031
 U 1 1 5C3516F5
 P 3650 3300
-F 0 "#PWR026" H 3650 3050 50  0001 C CNN
+F 0 "#PWR031" H 3650 3050 50  0001 C CNN
 F 1 "GND" H 3655 3127 50  0000 C CNN
 F 2 "" H 3650 3300 50  0001 C CNN
@@
 $EndComp
 $Comp
-L power:+3.3V #PWR025
+L power:+3.3V #PWR030
 U 1 1 5C351A76
 P 2400 2500
-F 0 "#PWR025" H 2400 2350 50  0001 C CNN
+F 0 "#PWR030" H 2400 2350 50  0001 C CNN
 F 1 "+3.3V" H 2415 2673 50  0000 C CNN
 F 2 "" H 2400 2500 50  0001 C CNN
@@
 Wire Wire Line
 	2300 3200 2800 3200
+$Comp
+L utsvt-bps:M24128 U4
+U 1 1 5F1359C0
+P 4250 2800
+F 0 "U4" H 4250 2965 50  0000 C CNN
+F 1 "M24128" H 4250 2874 50  0000 C CNN
+F 2 "Package_SO:SOIC-8_3.9x4.9mm_P1.27mm" H 4250 2800 50  0001 C CNN
+F 3 "https://www.st.com/resource/en/datasheet/m24128-bf.pdf" H 4250 2800 50  0001 C CNN
+F 4 "0x50" H 4250 2800 50  0001 C CNN "Address"
+	1    4250 2800
+	-1   0    0    -1
+$EndComp
 $EndSCHEMATC
